File: Asok75hotswap.kicad_pcb (KiCad board)
At the start: 2 copper layers, 314.8 x 141 mm, 224 parts, among them J1 AVR-ISP-6, SW1 SW_Push, U1 ATmega32U4-MU, U2 PRTR5V0U2X, Y1 16MHz

Commit message: Refactored project into two separate repositories
Other:
- outline, holes or cut-outs redrawn
- board text removed: "JLCJLCJLCJLC"
Changed lines of the file:
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@@
   (general
     (thickness 1.6)
-    (drawings 148)
+    (drawings 143)
     (tracks 3098)
     (zones 0)
@@
     )
   )
-  (gr_circle (center 274.6375 159.54375) (end 275.7895 159.54375) (layer Edge.Cuts) (width 0.05))
-  (gr_circle (center -35.71875 23.01875) (end -34.56675 23.01875) (layer Edge.Cuts) (width 0.05))
-  (gr_circle (center 274.6375 23.01875) (end 275.7895 23.01875) (layer Edge.Cuts) (width 0.05))
-  (gr_circle (center -34.925 159.54375) (end -33.773 159.54375) (layer Edge.Cuts) (width 0.05))
   (gr_text "Designed by Asok" (at 252.984 111.125) (layer B.SilkS)
     (effects (font (size 1 1) (thickness 0.15)) (justify mirror))
   )
-  (gr_text JLCJLCJLCJLC (at -29.464 154.813) (layer F.SilkS)
-    (effects (font (size 1 1) (thickness 0.15)))
-  )
   (gr_line (start 239.442665 152.129125) (end 218.755295 152.129125) (layer Edge.Cuts) (width 0.05))
